File: PCB/PCB.kicad_pcb (KiCad board)
At the start: 2 copper layers, 14 parts, among them M1 Motor_Servo, M2 Motor_Servo, SW1 RotaryEncoder_Switch, SW2 RotaryEncoder_Switch, SW3 SW_Push, SW4 SW_Push, SW5 SW_Push, SW6 SW_Push

Commit message: potato
Parts:
- added U1: XIAO-RP2040-DIP, Taranium-libs:XIAO-RP2040-DIP, F.Cu at (161.9, 76.2)
- D1, D2, D3, D4, D5, D6: moved to B.Cu
- moved SW6 81.6 mm to (183.5, 111.6)
- moved SW2 76.8 mm to (183.5, 90.4), turned to -90 degrees
- moved SW3 76.4 mm to (164.5, 92.6)
- moved SW5 70.0 mm to (164.5, 111.6)
- moved D1 69.2 mm to (172.4, 107.2)
- moved D6 68.5 mm to (171.4, 125.3), turned to 90 degrees
- moved SW4 65.7 mm to (145.4, 111.6)
- moved D5 54.8 mm to (152.4, 125.3), turned to 90 degrees
- moved SW1 54.4 mm to (145.4, 90.4), turned to -90 degrees
- moved M2 51.5 mm to (178.6, 69.1)
- moved D2 48.7 mm to (150.5, 107.2), turned to 180 degrees
- moved D3 46.6 mm to (152.4, 103.8), turned to 90 degrees
- moved D4 45.6 mm to (133.3, 125.3), turned to 90 degrees
- moved M1 23.3 mm to (145.3, 69.1)
Routing:
- net R2: track 0.00 -> 88.5 mm
- net GND: track 0.00 -> 73.5 mm
- net R1: track 0.00 -> 50.2 mm
- net C1: track 0.00 -> 39.7 mm
- net +5V: track 0.00 -> 37.6 mm
- net C3: track 0.00 -> 33.6 mm
- net C2: track 0.00 -> 32.8 mm
- net B1: track 0.00 -> 25.7 mm
- net A1: track 0.00 -> 20.5 mm
- net A2: track 0.00 -> 18.8 mm
- net B2: track 0.00 -> 13.5 mm
- net S2: track 0.00 -> 12.0 mm
- net S1: track 0.00 -> 9.25 mm
- net Net-(D6-A): track 0.00 -> 7.16 mm
- net Net-(D5-A): track 0.00 -> 7.16 mm
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Other:
- board outline added: 61.9 x 63.1 mm
