File: PCB/PCB.kicad_sch (KiCad schematic)
At the start: 15 parts, among them M1 Motor_Servo, M2 Motor_Servo, SW1 RotaryEncoder_Switch, SW2 RotaryEncoder_Switch, SW3 SW_Push, SW4 SW_Push, SW5 SW_Push, SW6 SW_Push, U1 XIAO-RP2040-DIP

Commit message: potato
Connections:
- net A1: now also U1.3 (P28_A2_D2); no longer U1.6 (P7_SCL_D5)
- net B1: now also U1.2 (P27_A1_D1); no longer U1.5 (P6_SDA_D4)
- net C1: now also U1.4 (P29_A3_D3); no longer U1.3 (P28_A2_D2)
- net R1: now also U1.6 (P7_SCL_D5); no longer U1.4 (P29_A3_D3)
- net R2: now also U1.5 (P6_SDA_D4); no longer U1.2 (P27_A1_D1)

Commit message: bleh
Parts:
- removed M1, M2: Motor_Servo, Connector_PinSocket_2.54mm:PinSocket_1x03_P2.54mm_Vertical, symbol Motor:Motor_Servo
Connections:
- net S1: no longer names the net of U1.1 (P26_A0_D0)
- net S2: no longer names the net of U1.11 (P3_D10_MOSI)
